Commit message: add spinner visuals

File: traj_opt/examples/spinner.urdf (robot description, URDF)
Before this commit: robot spinner, 3 links, 3 joints
Links:
- added link spinner, mass 1.0; visual box size=0.5 0.1 0.8; visual cylinder length=0.2 radius=.04
- link finger_two: geometry collision cylinder length=0.9 radius=.05; collision sphere radius=.05
Joints:
- added joint theta_three: type continuous, parent base, child spinner, origin xyz=1.0 0 1.0, axis 0 1 0

Commit message: simulate spinner system with contact, zero control inputs

File: traj_opt/examples/spinner.urdf (robot description, URDF)
Before this commit: robot spinner, 4 links, 4 joints
Links:
- link spinner: geometry collision box size=0.5 0.1 0.8; visual box size=0.5 0.1 0.8
Joints:
- joint theta_three: origin xyz=1.0 0 1.0 -> xyz=1.5 0 1.0

Commit message: make spinner thicker to avoid extraneous normal forces in the z direction

File: traj_opt/examples/spinner.urdf (robot description, URDF)
Before this commit: robot spinner, 4 links, 4 joints
Links:
- link finger_two: geometry collision sphere radius=.05; visual cylinder length=0.9 radius=.05
- link spinner: geometry collision box size=0.5 0.5 0.8; visual box size=0.5 0.5 0.8

Commit message: [WIP]: pushing sphere doesn't work as well as box

File: traj_opt/examples/spinner.urdf (robot description, URDF)
Before this commit: robot spinner, 4 links, 4 joints
Links:
- link spinner: geometry collision sphere radius=0.25; visual cylinder length=0.6 radius=.04

Commit message: add contact model parameters to yaml

File: traj_opt/examples/spinner.urdf (robot description, URDF)
Before this commit: robot spinner, 4 links, 4 joints
Links:
- link finger_one: geometry visual capsule length=0.9 radius=0.05
- link spinner: geometry collision box size=0.5 0.5 0.5; visual box size=0.5 0.5 0.5

Commit message: add cylinder example

File: traj_opt/examples/spinner.urdf (robot description, URDF)
Before this commit: robot spinner, 4 links, 4 joints
Links:
- link spinner: geometry collision cylinder length=0.6 radius=0.25; visual cylinder length=0.6 radius=.04
