Commit message: isolate similar bad convergence with one timestep

File: traj_opt/examples/spinner_capsule.urdf (robot description, URDF)
Before this commit: robot spinner, 4 links, 4 joints
Links:
- link finger_two: geometry collision capsule length=0.9 radius=0.05; collision sphere radius=.05

Commit message: avoid collision geometries with low precision signed distances

File: traj_opt/examples/spinner_capsule.urdf (robot description, URDF)
Before this commit: robot spinner, 4 links, 4 joints
Links:
- link finger_two: geometry collision sphere radius=.05; collision sphere radius=.05

File: traj_opt/examples/spinner_rectangle.urdf (robot description, URDF)
Before this commit: robot spinner, 4 links, 4 joints
Links:
- link finger_two: geometry collision sphere radius=.05; collision sphere radius=.05

File: traj_opt/examples/spinner_sphere.urdf (robot description, URDF)
Before this commit: robot spinner, 4 links, 4 joints
Links:
- link finger_two: geometry collision sphere radius=.05; collision sphere radius=.05

File: traj_opt/examples/spinner_square.urdf (robot description, URDF)
Before this commit: robot spinner, 4 links, 4 joints
Links:
- link finger_two: geometry collision sphere radius=.05; collision sphere radius=.05
