Commit message: add gflags option for spinner geometry

File: traj_opt/examples/spinner_sphere.urdf (robot description, URDF)
Before this commit: robot spinner, 4 links, 4 joints
Links:
- link finger_two: geometry collision cylinder length=0.9 radius=.05; collision sphere radius=.05

Commit message: Implements contact dissipation and friction.

File: traj_opt/examples/spinner_sphere.urdf (robot description, URDF)
Before this commit: robot spinner, 4 links, 4 joints
Links:
- link finger_two: geometry collision sphere radius=.05; visual cylinder length=0.9 radius=.05
- link spinner: geometry collision sphere radius=0.25; visual cylinder length=0.6 radius=.04

Commit message: analytical gradients improve wall-ball performance

File: traj_opt/examples/spinner_sphere.urdf (robot description, URDF)
Before this commit: robot spinner, 4 links, 4 joints
Links:
- link finger_two: geometry collision sphere radius=.05; visual cylinder length=0.9 radius=.05
